Commit message: Fixed gripper joint -  rbx1.urdf line 472 multiplier was incorrect (-1) changed to 1

File: rbx1_description/urdf/rbx1.urdf (robot description, URDF)
Before this commit: robot rbx1_description, 15 links, 14 joints
Joints:
- joint tip_gripper_idol_joint: mimic joint=gripper_idol_gear_joint multiplier=-1 offset=0 -> joint=gripper_idol_gear_joint multiplier=1 offset=0

Commit message: Robot base_link moved to origin in RViz simulation and gazebo so that coordinates are in reference to the base_link. Found new home pose after correction. Increased precision of get current pose.

File: rbx1_description/urdf/rbx1.urdf (robot description, URDF)
Before this commit: robot rbx1_description, 15 links, 14 joints
Joints:
- joint fixed: origin (none) -> xyz=0.2229 0.0923 0.04885 rpy=0 0 -1.178097

Commit message: Changed limits for gripper joints in urdf file to fix hand not working. The gripper hands can be set by one value that is set for both or seperate values for each side. Added capability for sepcifying the orientation of a pose by a facing vector and an angle of twist around this vector. This was added into the poseGoalClient.py file as a test for now but can later be implemented into the main code

File: rbx1_description/urdf/rbx1.urdf (robot description, URDF)
Before this commit: robot rbx1_description, 15 links, 14 joints
Joints:
- joint pivot_arm_gripper_idol_joint: limit lower=-1.5 upper=0 effort=5 velocity=1 -> lower=0 upper=1.5707 effort=5 velocity=1
- joint pivot_arm_gripper_servo_joint: limit lower=-1 upper=1 effort=5 velocity=1 -> lower=0 upper=1.5707 effort=5 velocity=1
- joint tip_gripper_idol_joint: limit lower=0 upper=1.4 effort=5 velocity=1 -> lower=0 upper=1.5707 effort=5 velocity=1
- joint tip_gripper_servo_joint: limit lower=0 upper=1.3 effort=5 velocity=1 -> lower=0 upper=1.5707 effort=5 velocity=1
